Commit message: Add warehouse SLAM A* workflow

File: src/px4_depth_description/urdf/x500_depth_down_tf.urdf (robot description, URDF)
Before this commit: robot x500_depth_down_tf, 4 links, 3 joints
Links:
- added link camera_rgb_frame
- added link camera_rgb_optical_frame
Joints:
- added joint camera_rgb_joint: type fixed, parent camera_link, child camera_rgb_frame, origin xyz=0 0 0 rpy=0 0 0
- added joint camera_rgb_optical_joint: type fixed, parent camera_rgb_frame, child camera_rgb_optical_frame, origin xyz=0 0 0 rpy=-1.5708 0 -1.5708
